File: sniffer-wifi/sniffer-wifi.kicad_sch (KiCad schematic)
At the start: 60 parts, among them J1 USB_B_Micro, J2 Conn_01x05_Socket, J3 Screw_Terminal_01x02, J4 Screw_Terminal_01x02, J5 Conn_02x04_Odd_Even, J6 flat number selector, Q1 MMBT3904, Q2 MMBT3904, Q5 MMBT3904, Q6 MMBT5551L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

Commit message: Add PCB design
Parts:
- removed C14, C7: 100n, symbol Device:C
- removed R10, R14, R15, R2, R20, R21, R22, R23, R4, R8: 10k, symbol Device:R
- removed R11, R12: 1k, Resistor_THT:R_Axial_DIN0207_L6.3mm_D2.5mm_P7.62mm_Horizontal, symbol Device:R
- removed U3: ATmega328PB, Package_QFP:TQFP-32_7x7mm_P0.8mm, symbol MCU_Microchip_ATmega:ATmega328P-A
- added C16: 100n, Capacitor_SMD:C_0805_2012Metric, symbol Device:C
- added RN2, RN3, RN4: 10k, Resistor_SMD:R_Array_Convex_4x0603, symbol Device:R_Pack04_Split
- added RN5: 1k, Resistor_SMD:R_Array_Convex_4x0603, symbol Device:R_Pack04_Split
- added U3: ATmega328PB, Package_QFP:TQFP-32_7x7mm_P0.8mm, symbol MCU_Microchip_ATmega:ATmega328PB-A
- C1, C10, C11, C15, C3, C5, C6, C9: footprint (none) -> Capacitor_SMD:C_0805_2012Metric
- C12: value 1n -> 100p; footprint (none) -> Capacitor_SMD:C_0805_2012Metric
- C13: value do not mount -> 1n; footprint (none) -> Capacitor_SMD:C_0805_2012Metric
- C2: footprint (none) -> Capacitor_SMD:CP_Elec_6.3x9.9
- C4, C8: footprint (none) -> Capacitor_SMD:C_1206_3216Metric
- D1: footprint (none) -> Diode_SMD:D_MiniMELF
- D4, D5: footprint LED_THT:LED_D3.0mm -> LED_SMD:LED_0805_2012Metric
- FB1, FB2, FB3, FB4: footprint (none) -> Inductor_SMD:L_0805_2012Metric
- J1: footprint Connector_USB:USB_Micro-AB_Molex_47590-0001 -> libs:USB_Micro-B
- J6: footprint Connector_IDC:IDC-Header_2x08_P2.54mm_Latch_Vertical -> Connector_PinHeader_2.54mm:PinHeader_2x08_P2.54mm_Vertical
- JP1: footprint (none) -> Connector_PinHeader_2.54mm:PinHeader_1x02_P2.54mm_Vertical
- R13, R16, R18: footprint (none) -> Resistor_SMD:R_0603_1608Metric
- R17, R19: footprint (none) -> Resistor_SMD:R_1206_3216Metric
- R3: footprint Resistor_THT:R_Axial_DIN0207_L6.3mm_D2.5mm_P7.62mm_Horizontal -> Resistor_SMD:R_1206_3216Metric
- R5, R7, R9: footprint (none) -> Resistor_SMD:R_0805_2012Metric
Connections:
- net +3V3: now also RN2.1 (R1.1), RN2.2 (R2.1), RN2.3 (R3.1), RN3.1 (R1.1), RN3.2 (R2.1), RN3.3 (R3.1), RN4.2 (R2.1), RN4.3 (R3.1)
- net +5V: now also C11.1, RN2.4 (R4.1), RN4.1 (R1.1), U3.4 (VCC)
- net ADC: now also U3.23 (PC0)
- net AVCC: now also U3.18 (AVCC)
- net CH_PD: now also RN4.6 (R3.2)
- net ESP_RESET: now also C16.1, RN2.7 (R2.2); no longer C11.1
- net ESP_RX: now also RN4.7 (R2.2)
- net F0: now also U3.25 (PC2)
- net F1: now also U3.26 (PC3)
- net F2: now also U3.27 (PC4)
- net F3: now also U3.28 (PC5)
- net F4: now also U3.2 (PD4)
- net F5: now also U3.9 (PD5)
- net F6: now also U3.10 (PD6)
- net F7: now also U3.11 (PD7)
- net GND: now also C16.2, U3.21 (GND), U3.5 (GND)
- net GPIO0: now also RN2.8 (R1.2)
- net GPIO2: now also RN2.6 (R3.2)
- net L+TTL: now also U3.1 (PD3), U3.32 (PD2)
- net MISO: now also U3.16 (PB4)
- net MOSI: now also U3.15 (PB3)
- net PD_CONTROL: now also U3.14 (PB2)
- net RESET: now also RN2.5 (R4.2), U3.29 (~{RESET}/PC6)
- net RXD: now also RN4.8 (R1.2), U3.30 (PD0)
- net SCK: now also U3.17 (PB5)
- net STATUS_GREEN: now also RN5.8 (R1.2), U3.12 (PB0)
- net STATUS_RED: now also RN5.7 (R2.2), U3.13 (PB1)
- net TXD: now also U3.31 (PD1)
- net XTAL1: now also U3.7 (XTAL1/PB6)
- net XTAL2: now also U3.8 (XTAL2/PB7)
- net at D5.1 (K): now also RN5.2 (R2.1)
- net at Q1.1 (B): now also RN3.6 (R3.2)
- net at C6.1: now also U3.20 (AREF)
- net at Q5.1 (B): now also RN3.8 (R1.2)
- net at Q2.1 (B): now also RN3.7 (R2.2)
- net at D4.1 (K): now also RN5.1 (R1.1)
- no-connect marks 6 -> 8
Other:
- moved on the sheet: C12, D1, D6, R3
